Commit message: update: add visualization tool

File: examples/world_engine/piper_description/urdf/piper_description.urdf (robot description, URDF)
Before this commit: robot piper_description, 9 links, 8 joints
Links:
- link base_link: geometry collision mesh filename=../meshes/base_link.STL; visual mesh filename=../meshes/base_link.dae
- link link1: geometry collision mesh filename=../meshes/link1.STL; visual mesh filename=../meshes/link1.dae
- link link2: geometry collision mesh filename=../meshes/link2.STL; visual mesh filename=../meshes/link2.dae
- link link3: geometry collision mesh filename=../meshes/link3.STL; visual mesh filename=../meshes/link3.dae
- link link4: geometry collision mesh filename=../meshes/link4.STL; visual mesh filename=../meshes/link4.dae
- link link5: geometry collision mesh filename=../meshes/link5.STL; visual mesh filename=../meshes/link5.dae
- link link6: geometry collision mesh filename=../meshes/link6_1.STL; visual mesh filename=../meshes/link6.dae
- link link7: geometry collision mesh filename=../meshes/link7.STL; visual mesh filename=../meshes/link7.dae
- link link8: geometry collision mesh filename=../meshes/link8.STL; visual mesh filename=../meshes/link8.dae
